Commit message: My changes in the submodule

File: pmb2_description/robots/pmb2.urdf.xacro (robot description, xacro)
@@ -15,7 +15,7 @@
   <!-- ARGUMENTS -->
   <!-- no-laser, hokuyo, sick-551, sick-561, sick-571-->
-  <xacro:arg name="laser_model" default="sick-571"/>
+  <xacro:arg name="laser_model" default="no-laser"/>
   <!-- false, true -->
-  <xacro:arg name="has_sonars" default="true"/>
+  <xacro:arg name="has_sonars" default="false"/>
   <!-- false, true -->
   <xacro:arg name="has_microphone" default="false"/>
@@ -30,9 +30,9 @@
   <!-- PROPERTIES -->
   <!-- HW configuration -->
-  <xacro:property name="laser_model" value="$(arg laser_model)" />
-  <xacro:property name="has_sonars" value="$(arg has_sonars)" />
-  <xacro:property name="has_microphone" value="$(arg has_microphone)" />
-  <xacro:property name="add_on_module" value="$(arg add_on_module)"/>
-  <xacro:property name="camera_model" value="$(arg camera_model)" />
+  <xacro:property name="laser_model" value="no-laser" />
+  <xacro:property name="has_sonars" value="false" />
+  <xacro:property name="has_microphone" value="false" />
+  <xacro:property name="add_on_module" value="no-add-on"/>
+  <xacro:property name="camera_model" value="no-camera" />
   <!-- HW configuration check -->
   <xacro:if value="${laser_model not in ['no-laser', 'sick-551', 'sick-561', 'sick-571', 'hokuyo']}">

File: pmb2_description/ros2_control/ros2_control.urdf.xacro (robot description, xacro)
@@ -20,5 +20,5 @@
     <xacro:if value="${use_sim_time}">
       <gazebo>
-        <plugin filename="libgazebo_ros2_control.so" name="gazebo_ros2_control">
+        <plugin filename="libgz_ros2_control-system.so" name="gz_ros2_control::GazeboSimROS2ControlPlugin">
           <ros>
             <namespace>${namespace}</namespace>
@@ -36,5 +36,5 @@
         <!-- HW interface gazebo-->
         <hardware>
-          <plugin>gazebo_ros2_control/GazeboSystem</plugin>
+          <plugin>gz_ros2_control/GazeboSimSystem</plugin>
         </hardware>
       </xacro:if>

File: pmb2_description/urdf/base/base.gazebo.xacro (robot description, xacro)
@@ -32,12 +32,12 @@
     <!-- Odometry plugin for ground truth -->
     <gazebo>
-      <plugin filename="libgazebo_world_odometry.so" name="gazebo_ros_odometry">
-        <ros>
-          <namespace>${namespace}</namespace>
-        </ros>
-        <frame_name>world</frame_name>
-        <body_name>base_footprint</body_name>
-        <topic_name>ground_truth_odom</topic_name>
-        <update_rate>100.0</update_rate>
+      <plugin filename="libgz-sim8-odometry-publisher-system.so"
+              name="gz::sim::systems::OdometryPublisher">
+        <publish_tf>true</publish_tf>
+        <link_name>pmb2::base_footprint</link_name>    <!-- the robot link to track -->
+        <odom_frame>odom</odom_frame>
+        <robot_base_frame>base_footprint</robot_base_frame>
+        <publish_rate>50</publish_rate>        <!-- Hz -->
+        <use_sim_time>true</use_sim_time>
       </plugin>
     </gazebo>

File: pmb2_description/urdf/wheels/caster.gazebo.xacro (robot description, xacro)
@@ -21,5 +21,5 @@
       <kd>100.0</kd>
       <minDepth>0.002</minDepth>
-      <maxVel>1.0</maxVel>
+      <maxVel>3.0</maxVel>
       <material>Gazebo/DarkGrey</material>
     </gazebo>

File: pmb2_description/urdf/wheels/wheel.gazebo.xacro (robot description, xacro)
@@ -21,5 +21,5 @@
       <kd>100.0</kd>
       <minDepth>0.002</minDepth>
-      <maxVel>1.0</maxVel>
+      <maxVel>3.0</maxVel>
       <material>Gazebo/DarkGrey</material>
     </gazebo>

File: pmb2_description/urdf/wheels/wheel.ros2_control.xacro (robot description, xacro)
@@ -18,4 +18,5 @@
       <command_interface name="velocity" />
       <state_interface name="position" />
+      <state_interface name="velocity" />
     </joint>
     <transmission name="wheel_${side}_trans">
